File: Kicad/Placa_carro/Placa_carro.kicad_pcb (KiCad board)
At the start: 2 copper layers, 4 parts, among them J1 Conn_01x19, J2 Conn_01x19, U1 PIC16F887-IP, U2 L293D

Commit message: Terminada placa motores
Parts:
- removed U2: L293D, Package_DIP:DIP-16_W7.62mm
- added J3: ADXL345, Connector_PinSocket_2.54mm:PinSocket_1x08_P2.54mm_Vertical, F.Cu at (147.3, 40.6)
- added J4: Servo, Connector_PinHeader_2.54mm:PinHeader_1x03_P2.54mm_Vertical, F.Cu at (154.9, 48.3)
- added J5: Conn_01x06, Connector_PinSocket_2.54mm:PinSocket_1x06_P2.54mm_Vertical, F.Cu at (147.3, 68.6)
- added R1: R_US, Resistor_THT:R_Axial_DIN0309_L9.0mm_D3.2mm_P12.70mm_Horizontal, F.Cu at (156.2, 73.7)
- added R2: R_US, Resistor_THT:R_Axial_DIN0309_L9.0mm_D3.2mm_P12.70mm_Horizontal, F.Cu at (156.2, 78.4)
- added Slave1: PIC16F887-IP, Package_DIP:DIP-40_W15.24mm, F.Cu at (101.6, 40.6)
- J1: value Conn_01x19 -> Motor_signal; footprint Connector_PinSocket_2.54mm:PinSocket_1x19_P2.54mm_Vertical -> TerminalBlock:TerminalBlock_bornier-2_P5.08mm
- J2: value Conn_01x19 -> VOLT; footprint Connector_PinSocket_2.54mm:PinSocket_1x19_P2.54mm_Vertical -> TerminalBlock:TerminalBlock_bornier-2_P5.08mm
- moved J2 42.0 mm to (162.6, 86.4)
- moved J1 22.7 mm to (167.6, 55.9)
- moved Master1 14.1 mm to (124.5, 41.9)
- renumbered U1 to Master1
Connections:
- net /D6 renamed /M1
- net /D7 renamed /M2
- J2 pad 1: /5V -> /VDD
- Master1 pad 18: unconnected-(U1-SCL/SCK/RC3-Pad18) -> /SCL
- Master1 pad 23: unconnected-(U1-SDA/SDI/RC4-Pad23) -> /SDA
- Master1 pad 25: unconnected-(U1-TX/CK/RC6-Pad25) -> /RX
- Master1 pad 26: unconnected-(U1-RX/DT/RC7-Pad26) -> /TX

Commit message: Terminada la placa del carro
Parts:
- J5: value Conn_01x06 -> HC-05
- moved J1 99.2 mm to (91.4, 119.4)
- moved J3 97.0 mm to (78.7, 109.2), turned to 180 degrees
- moved R2 81.4 mm to (83.8, 115.6), turned to 90 degrees
- moved R1 72.4 mm to (83.8, 72.4), turned to -90 degrees
- moved Slave1 69.1 mm to (142.2, 96.5), turned to -90 degrees
- moved J4 57.5 mm to (114.3, 88.9), turned to 90 degrees
- moved J2 45.2 mm to (127.0, 58.4), turned to -90 degrees
- moved Master1 30.5 mm to (94.0, 40.6)
- moved J5 17.0 mm to (132.1, 76.2), turned to -90 degrees
Connections:
- Master1 pad 11: unconnected-(Master1-VDD-Pad11) -> /VDD
- Master1 pad 12: unconnected-(Master1-VSS-Pad12) -> /GND
- Master1 pad 31: unconnected-(Master1-VSS-Pad31) -> /GND
- Master1 pad 32: unconnected-(Master1-VDD-Pad32) -> /VDD
- Slave1 pad 11: unconnected-(Slave1-VDD-Pad11) -> /VDD
- Slave1 pad 12: unconnected-(Slave1-VSS-Pad12) -> /GND
- Slave1 pad 17: unconnected-(Slave1-P1A/CCP1/RC2-Pad17) -> /SGN
- Slave1 pad 21: unconnected-(Slave1-RD2-Pad21) -> /M1
- Slave1 pad 22: unconnected-(Slave1-RD3-Pad22) -> /M2
- Slave1 pad 31: unconnected-(Slave1-VSS-Pad31) -> /GND
- Slave1 pad 32: unconnected-(Slave1-VDD-Pad32) -> /VDD
Routing:
- net /VDD: track 0.00 -> 157.2 mm
- net /SDA: track 0.00 -> 131.6 mm
- net /GND: track 0.00 -> 118.9 mm
- net /SCL: track 0.00 -> 37.0 mm
- net /SGN: track 0.00 -> 22.4 mm
- net /TX: track 0.00 -> 17.3 mm
- net /RX: track 0.00 -> 13.8 mm
- net /M1: track 0.00 -> 8.68 mm
- net /M2: track 0.00 -> 7.62 mm
Other:
- board outline added: 96.5 x 99.1 mm

Commit message: Avances varios
Terminada la placa del carro
Pruebas avanzadas del esclavo
Parts:
- added J6: 3Vreg, Connector_PinHeader_2.54mm:PinHeader_1x03_P2.54mm_Vertical, F.Cu at (116.8, 63.5)
- added J7: HC89_1, Connector_PinHeader_2.54mm:PinHeader_1x03_P2.54mm_Vertical, F.Cu at (124.5, 116.8)
- added J8: HC89_2, Connector_PinHeader_2.54mm:PinHeader_1x03_P2.54mm_Vertical, F.Cu at (139.7, 114.3)
- moved J4 5.68 mm to (116.8, 83.8)
- moved J1 5.68 mm to (94.0, 114.3)
- moved J3 5.68 mm to (81.3, 104.1)
- moved R1 5.68 mm to (86.4, 67.3)
- moved R2 5.68 mm to (86.4, 110.5)
- moved J2 5.68 mm to (129.5, 53.3)
- moved J5 5.68 mm to (134.6, 71.1)
- moved Master1 5.68 mm to (96.5, 35.6)
- moved Slave1 5.68 mm to (144.8, 91.4)
Connections:
- J3 pad 2: /VCC -> /3V
- J5 pad 2: /VDD -> /3V
- Slave1 pad 33: unconnected-(Slave1-INT/AN12/RB0-Pad33) -> /HC89
- Slave1 pad 34: unconnected-(Slave1-C12IN3-/AN10/RB1-Pad34) -> /HC89_2
Routing:
- net /3V: track 0.00 -> 184.7 mm, vias 0 -> 4
- net /GND: track 118.9 -> 298.1 mm, vias 0 -> 4
- net /VDD: track 157.2 -> 307.4 mm, vias 0 -> 4
- net /HC89_2: track 0.00 -> 12.3 mm
- net /HC89: track 0.00 -> 10.2 mm
- net /SDA: track 131.6 -> 138.2 mm
