File: Kicad/Placa_carro/Placa_carro.kicad_sch (KiCad schematic)
At the start: 5 parts, among them J1 ESP izq, J2 ESP der, J3 ADXL345, U1 PIC16F887-IP, U2 L293D

Commit message: Terminada placa motores
Parts:
- removed J1: ESP izq, Connector_PinSocket_2.54mm:PinSocket_1x19_P2.54mm_Vertical, symbol Conect_gen:Conn_01x19
- removed J2: ESP der, Connector_PinSocket_2.54mm:PinSocket_1x19_P2.54mm_Vertical, symbol Conect_gen:Conn_01x19
- removed U2: L293D, Package_DIP:DIP-16_W7.62mm, symbol Driver_Motor:L293D
- added J1: Motor_signal, TerminalBlock:TerminalBlock_bornier-2_P5.08mm, symbol Connector:Screw_Terminal_01x02
- added J2: VOLT, TerminalBlock:TerminalBlock_bornier-2_P5.08mm, symbol Connector:Screw_Terminal_01x02
- added J4: Servo, Connector_PinHeader_2.54mm:PinHeader_1x03_P2.54mm_Vertical, symbol Conect_gen:Conn_01x03
- added J5: Conn_01x06, Connector_PinSocket_2.54mm:PinSocket_1x06_P2.54mm_Vertical, symbol Conect_gen:Conn_01x06
- added R1, R2: R_US, Resistor_THT:R_Axial_DIN0309_L9.0mm_D3.2mm_P12.70mm_Horizontal, symbol Device:R_US
- added Slave1: PIC16F887-IP, Package_DIP:DIP-40_W15.24mm, symbol MCU_Microchip_PIC16:PIC16F887-IP
- J3: footprint (none) -> Connector_PinSocket_2.54mm:PinSocket_1x08_P2.54mm_Vertical
- renumbered U1 to Master1
Connections:
- net EN: now also J5.1 (Pin_1)
- net GND: now also J2.2 (Pin_2), J4.1 (Pin_1), J5.3 (Pin_3)
- net SCL: now also Master1.18 (SCL/SCK/RC3), R1.2, Slave1.18 (SCL/SCK/RC3)
- net SDA: now also Master1.23 (SDA/SDI/RC4), R2.2, Slave1.23 (SDA/SDI/RC4)
- net RX: now reaches Master1.25 (TX/CK/RC6)
- net RX: now also J5.5 (Pin_5)
- net TX: now reaches Master1.26 (RX/DT/RC7)
- net TX: now also J5.4 (Pin_4)
- new net M1: J1.1 (Pin_1)
- new net M2: J1.2 (Pin_2)
- new net SGN: J4.3 (Pin_3)
- new net STATE: J5.6 (Pin_6)
- new net VDD: J2.1 (Pin_1), J4.2 (Pin_2), J5.2 (Pin_2), R1.1, R2.1

Commit message: Terminada la placa del carro
Parts:
- J5: value Conn_01x06 -> HC-05
Connections:
- net GND: now also Master1.12 (VSS), Master1.31 (VSS), Slave1.12 (VSS), Slave1.31 (VSS)
- net M1: now also Slave1.21 (RD2)
- net M2: now also Slave1.22 (RD3)
- net SGN: now also Slave1.17 (P1A/CCP1/RC2)
- net VDD: now also Master1.11 (VDD), Master1.32 (VDD), Slave1.11 (VDD), Slave1.32 (VDD)
Changed lines of the file:
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@@
 (kicad_sch (version 20230121) (generator eeschema)
   (paper "A4")
+  (junction (at 137.16 187.96) (diameter 0) (color 0 0 0 0)
+  )
+  (junction (at 148.59 100.33) (diameter 0) (color 0 0 0 0)
+  )
   (wire (pts (xy 73.66 54.61) (xy 77.47 54.61))
     (stroke (width 0) (type default))
@@
     (stroke (width 0) (type default))
   )
+  (wire (pts (xy 137.16 104.14) (xy 137.16 107.95))
+    (stroke (width 0) (type default))
+  )
   (wire (pts (xy 67.31 118.11) (xy 71.12 118.11))
     (stroke (width 0) (type default))
@@
     (stroke (width 0) (type default))
   )
+  (wire (pts (xy 139.7 104.14) (xy 139.7 107.95))
+    (stroke (width 0) (type default))
+  )
+  (wire (pts (xy 167.64 161.29) (xy 170.18 161.29))
+    (stroke (width 0) (type default))
+  )
   (wire (pts (xy 176.53 87.63) (xy 180.34 87.63))
     (stroke (width 0) (type default))
   )
+  (wire (pts (xy 148.59 100.33) (xy 153.67 100.33))
+    (stroke (width 0) (type default))
+  )
   (wire (pts (xy 73.66 52.07) (xy 77.47 52.07))
     (stroke (width 0) (type default))
@@
     (stroke (width 0) (type default))
   )
+  (wire (pts (xy 146.05 20.32) (xy 148.59 20.32))
+    (stroke (width 0) (type default))
+  )
+  (wire (pts (xy 137.16 187.96) (xy 135.89 187.96))
+    (stroke (width 0) (type default))
+  )
+  (wire (pts (xy 106.68 140.97) (xy 111.76 140.97))
+    (stroke (width 0) (type default))
+  )
   (wire (pts (xy 208.28 68.58) (xy 208.28 62.23))
     (stroke (width 0) (type default))
@@
     (stroke (width 0) (type default))
   )
+  (wire (pts (xy 146.05 100.33) (xy 148.59 100.33))
+    (stroke (width 0) (type default))
+  )
+  (wire (pts (xy 146.05 24.13) (xy 146.05 20.32))
+    (stroke (width 0) (type default))
+  )
+  (wire (pts (xy 139.7 184.15) (xy 139.7 187.96))
+    (stroke (width 0) (type default))
+  )
   (wire (pts (xy 167.64 163.83) (xy 175.26 163.83))
     (stroke (width 0) (type default))
   )
+  (wire (pts (xy 148.59 20.32) (xy 148.59 24.13))
+    (stroke (width 0) (type default))
+  )
   (wire (pts (xy 67.31 107.95) (xy 71.12 107.95))
     (stroke (width 0) (type default))
@@
     (stroke (width 0) (type default))
   )
+  (wire (pts (xy 137.16 184.15) (xy 137.16 187.96))
+    (stroke (width 0) (type default))
+  )
+  (wire (pts (xy 153.67 101.6) (xy 153.67 100.33))
+    (stroke (width 0) (type default))
+  )
   (wire (pts (xy 208.28 76.2) (xy 208.28 80.01))
     (stroke (width 0) (type default))
   )
+  (wire (pts (xy 106.68 138.43) (xy 111.76 138.43))
+    (stroke (width 0) (type default))
+  )
+  (wire (pts (xy 139.7 187.96) (xy 137.16 187.96))
+    (stroke (width 0) (type default))
+  )
   (wire (pts (xy 194.31 62.23) (xy 194.31 68.58))
     (stroke (width 0) (type default))
@@
     (stroke (width 0) (type default))
   )
+  (wire (pts (xy 137.16 104.14) (xy 139.7 104.14))
+    (stroke (width 0) (type default))
+  )
   (wire (pts (xy 67.31 86.36) (xy 71.12 86.36))
     (stroke (width 0) (type default))
@@
     (stroke (width 0) (type default))
   )
+  (label "M2" (at 106.68 140.97 180) (fields_autoplaced)
+    (effects (font (size 1.27 1.27)) (justify right bottom))
+  )
   (label "INT2" (at 67.31 110.49 0) (fields_autoplaced)
     (effects (font (size 1.27 1.27)) (justify left bottom))
@@
     (effects (font (size 1.27 1.27)) (justify right bottom))
   )
+  (label "M1" (at 106.68 138.43 180) (fields_autoplaced)
+    (effects (font (size 1.27 1.27)) (justify right bottom))
+  )
   (label "RX" (at 180.34 87.63 0) (fields_autoplaced)
     (effects (font (size 1.27 1.27)) (justify left bottom))
@@
     (effects (font (size 1.27 1.27)) (justify left bottom))
   )
+  (label "VDD" (at 137.16 104.14 180) (fields_autoplaced)
+    (effects (font (size 1.27 1.27)) (justify right bottom))
+  )
+  (label "VDD" (at 147.32 20.32 90) (fields_autoplaced)
+    (effects (font (size 1.27 1.27)) (justify left bottom))
+  )
   (label "VDD" (at 95.25 78.74 180) (fields_autoplaced)
     (effects (font (size 1.27 1.27)) (justify right bottom))
@@
     (effects (font (size 1.27 1.27)) (justify left bottom))
   )
+  (label "GND" (at 135.89 187.96 180) (fields_autoplaced)
+    (effects (font (size 1.27 1.27)) (justify right bottom))
+  )
   (label "GND" (at 67.31 100.33 0) (fields_autoplaced)
     (effects (font (size 1.27 1.27)) (justify left bottom))
@@
     (effects (font (size 1.27 1.27)) (justify right bottom))
   )
+  (label "GND" (at 153.67 101.6 0) (fields_autoplaced)
+    (effects (font (size 1.27 1.27)) (justify left bottom))
+  )
   (label "SDA" (at 208.28 80.01 270) (fields_autoplaced)
     (effects (font (size 1.27 1.27)) (justify right bottom))
@@
   )
   (label "SDA" (at 67.31 115.57 0) (fields_autoplaced)
+    (effects (font (size 1.27 1.27)) (justify left bottom))
+  )
+  (label "SGN" (at 170.18 161.29 0) (fields_autoplaced)
     (effects (font (size 1.27 1.27)) (justify left bottom))
   )
@@
       (effects (font (size 1.27 1.27)) (justify left))
     )
-    (property "Value" "Conn_01x06" (at 106.68 83.82 0)
-      (effects (font (size 1.27 1.27)) (justify left))
-    )
+    (property "Value" "HC-05" (at 106.68 83.82 0)
+      (effects (font (size 1.27 1.27)) (justify left))
+    )

Commit message: Avances varios
Terminada la placa del carro
Pruebas avanzadas del esclavo
Parts:
- added J6: 3Vreg, Connector_PinHeader_2.54mm:PinHeader_1x03_P2.54mm_Vertical, symbol Conect_gen:Conn_01x03
- added J7: HC89_1, Connector_PinHeader_2.54mm:PinHeader_1x03_P2.54mm_Vertical, symbol Conect_gen:Conn_01x03
- added J8: HC89_2, Connector_PinHeader_2.54mm:PinHeader_1x03_P2.54mm_Vertical, symbol Conect_gen:Conn_01x03
Connections:
- net GND: now also J6.1 (Pin_1), J7.1 (Pin_1), J8.1 (Pin_1)
- net VDD: now also J6.2 (Pin_2), J7.3 (Pin_3), J8.3 (Pin_3); no longer J5.2 (Pin_2)
- net HC89: now reaches Slave1.33 (INT/AN12/RB0)
- net HC89: now also J7.2 (Pin_2)
- net HC89_2: now reaches Slave1.34 (C12IN3-/AN10/RB1)
- net HC89_2: now also J8.2 (Pin_2)
- net VCC renamed 3V
- net 3V: now also J5.2 (Pin_2), J6.3 (Pin_3)
